Commit message: Refactor RoboMapperNode and VisionNode for improved functionality and parameterization
- Enhanced RoboMapperNode with dynamic parameter loading for map configuration (topic names, resolution, dimensions, and publish rate).
- Implemented ray casting algorithm in RoboMapperNode for better obstacle detection and mapping.
- Improved logging messages for better clarity and debugging.
- Updated VisionNode to include dynamic parameterization for color detection thresholds and added debug visualization options.
- Refactored image processing logic in VisionNode to improve clarity and maintainability.
- Changed file permissions for test_gripper.py to ensure proper execution.

File: description/robot.urdf.xacro (robot description, xacro)
@@ -65,7 +65,7 @@
     <xacro:box_inertia m="0" w="0" d="0" h="0"/>
     <joint name="base_footprint_joint" type="fixed">
-      <parent link="base_footprint"/>
-      <child link="base_link"/>
-      <origin xyz="0 0 0.05" rpy="0 0 0"/>
+      <parent link="base_link"/>
+      <child link="base_footprint"/>
+      <origin xyz="0 0 -0.05" rpy="0 0 0"/>
     </joint>
   </link>

Commit message: feat: Update path planning and state machine logic for improved obstacle handling and pathfinding efficiency

File: description/robot.urdf.xacro (robot description, xacro)
@@ -67,5 +67,5 @@
       <parent link="base_link"/>
       <child link="base_footprint"/>
-      <origin xyz="0 0 -0.05" rpy="0 0 0"/>
+      <origin xyz="0 0 0" rpy="0 0 0"/> <!-- Centro deve estar no meio -->
     </joint>
   </link>
